Commit message: fixed front right wheel collision radius to match visual size

File: description/robot_core.xacro (robot description, xacro)
@@ -85,5 +85,5 @@
         <collision>
             <geometry>
-                <sphere radius="0.05" />
+                <sphere radius="0.0425" />
             </geometry>
             <material name="blue"/>
