Commit message: Apply Joan's updates to correct directory structure

File: robot2_ws/src/my_robot/description/lidar.xacro (robot description, xacro)
@@ -25,5 +25,5 @@
     </xacro:inertial_cylinder>
   </link>
-  <!-- GAZEBO GPU LIDAR SENSOR CONFIGURATION -->
+  <!-- GAZEBO LIDAR SENSOR CONFIGURATION -->
   <gazebo reference="laser_frame">
     <sensor name="laser" type="gpu_lidar">
@@ -48,9 +48,3 @@
     </sensor>
   </gazebo>
-  <!-- GAZEBO SENSORS SYSTEM PLUGIN -->
-  <gazebo>
-    <plugin filename="gz-sim-sensors-system" name="gz::sim::systems::Sensors">
-      <render_engine>ogre2</render_engine>
-    </plugin>
-  </gazebo>
 </robot>

File: robot2_ws/src/my_robot/description/robot_core.xacro (robot description, xacro)
@@ -79,5 +79,5 @@
         <visual>
             <geometry>
-                <cylinder length="0.031" radius="0.05" />
+                <cylinder length="0.031" radius="0.0425" />
             </geometry>
             <material name="blue"/>
@@ -85,5 +85,5 @@
         <collision>
             <geometry>
-                <sphere radius="0.05" />
+                <sphere radius="0.0425" />
             </geometry>
             <material name="blue"/>
@@ -93,5 +93,5 @@
         </xacro:inertial_cylinder>
     </link>
-    <gazebo reference="front_left_wheel">
+    <gazebo reference="front_right_wheel">
     </gazebo>
     <!-- BACK LEFT WHEEL -->
